File: EAGLE/projects/nRF_board.brd (EAGLE design)
At the start: 50 x 50 mm, 18 parts

Commit message: nRF_board
Parts:
- moved C2 1.27 mm to (45.7, 33.0)
- moved C6 1.27 mm to (45.7, 7.62)
- moved JP2 1.27 mm to (36.8, 33.0)
- moved JP3 1.27 mm to (36.8, 7.62)
- turned C3 to 90 degrees
- turned C7 to 90 degrees
Routing:
- net +3V3: track 120.2 -> 122.3 mm
- net N$15: track 3.59 -> 1.80 mm
- net N$9: track 34.0 -> 35.3 mm
- net N$8: track 29.3 -> 30.6 mm
- net N$6: track 47.0 -> 48.3 mm
- net N$5: track 26.8 -> 28.0 mm
- net N$4: track 29.3 -> 30.6 mm
- net N$14: track 29.3 -> 30.6 mm
- net N$12: track 47.0 -> 48.3 mm
- net N$10: track 29.3 -> 30.6 mm
- net N$7: track 31.8 -> 33.1 mm
- net N$13: track 31.8 -> 33.1 mm
- net N$11: track 26.8 -> 28.0 mm
- net N$2: track 34.0 -> 35.3 mm
- net GND: track 127.6 -> 128.3 mm
